File: pcb/otukset/otukset.kicad_sch (KiCad schematic)
At the start: 0 parts

Commit message: stuff
Parts:
- added C1, C2, C3: C, Capacitor_SMD:C_0805_2012Metric, symbol Device:C
- added SW1: RotaryEncoder_Switch, EC11:EC11_Horizontal, symbol Device:RotaryEncoder_Switch
- added U1: ESP32C5, ESP32C5:ESP32C5, symbol ESP32C5:ESP32C5
- added U2: GM803, GM803:GM803, symbol GM803:GM803
- added U3: 240x320_ST7789, 240x320_ST7789:240x320_ST7789_2.8, symbol 240x320_ST7789:240x320_ST7789
- added U4: BMI160, BMI160:BMI160, symbol BMI160:BMI160
Connections:
- new net +3.3V: C1.1, C2.1, C3.1, U1.2 (3V3), U2.2 (VCC), U3.1 (VCC), U4.1 (VIN), U4.2 (3V3)
- new net GND: C1.2, C2.2, C3.2, U1.1 (GND), U1.28 (GND), U2.3 (GND), U3.2 (GND), U4.3 (GND)
- new net SCAN_RX: U1.16 (IO5), U2.4 (RXD)
- new net SCAN_SUCCESS: U1.18 (IO27), U2.10 (LED3)
- new net SCAN_TX: U1.17 (IO4), U2.5 (TXD)
- new net ~{SCAN_TRIG}: U1.15 (IO28), U2.12 (TRIG)
